Commit message: Replaced RoboMaker source code with latest version

File: simulation/aws-robomaker-sample-application-deepracer/simulation_ws/src/deepracer_simulation/urdf/mit/macros.xacro (robot description, xacro)
@@ -34,5 +34,5 @@
   <origin xyz="0 0 0" rpy="0 0 0" />
   <geometry>
-      <mesh scale="0.6 0.6 0.6" filename="package://deepracer_simulation/meshes/chassis.STL"/>
+      <mesh scale="0.6 0.6 0.6" filename="package://deepracer_simulation/meshes/mit/chassis.STL"/>
   </geometry>
 </xacro:macro>
@@ -40,5 +40,5 @@
   <origin xyz="0 0 0" rpy="0 0 0" />
   <geometry>
-    <mesh scale="0.6 0.6 0.6" filename="package://deepracer_simulation/meshes/left_rear_wheel.STL" />
+    <mesh scale="0.6 0.6 0.6" filename="package://deepracer_simulation/meshes/mit/left_rear_wheel.STL" />
   </geometry>
 </xacro:macro>
@@ -46,5 +46,5 @@
   <origin xyz="0 0 0" rpy="0 0 0" />
   <geometry>
-    <mesh scale="0.6 0.6 0.6" filename="package://deepracer_simulation/meshes/right_rear_wheel.STL" />
+    <mesh scale="0.6 0.6 0.6" filename="package://deepracer_simulation/meshes/mit/right_rear_wheel.STL" />
   </geometry>
 </xacro:macro>
@@ -52,5 +52,5 @@
   <origin xyz="0 0 0" rpy="0 0 0" />
   <geometry>
-    <mesh scale="0.6 0.6 0.6" filename="package://deepracer_simulation/meshes/left_front_wheel.STL" />
+    <mesh scale="0.6 0.6 0.6" filename="package://deepracer_simulation/meshes/mit/left_front_wheel.STL" />
   </geometry>
 </xacro:macro>
@@ -58,5 +58,5 @@
   <origin xyz="0 0 0" rpy="0 0 0" />
   <geometry>
-    <mesh scale="0.6 0.6 0.6" filename="package://deepracer_simulation/meshes/right_front_wheel.STL" />
+    <mesh scale="0.6 0.6 0.6" filename="package://deepracer_simulation/meshes/mit/right_front_wheel.STL" />
   </geometry>
 </xacro:macro>
@@ -64,5 +64,5 @@
   <origin xyz="0 0 0" rpy="0 0 0" />
   <geometry>
-    <mesh scale="0.6 0.6 0.6" filename="package://deepracer_simulation/meshes/left_steering_hinge.STL" />
+    <mesh scale="0.6 0.6 0.6" filename="package://deepracer_simulation/meshes/mit/left_steering_hinge.STL" />
   </geometry>
 </xacro:macro>
@@ -70,5 +70,5 @@
   <origin xyz="0 0 0" rpy="0 0 0" />
   <geometry>
-    <mesh scale="0.6 0.6 0.6" filename="package://deepracer_simulation/meshes/right_steering_hinge.STL" />
+    <mesh scale="0.6 0.6 0.6" filename="package://deepracer_simulation/meshes/mit/right_steering_hinge.STL" />
   </geometry>
 </xacro:macro>

File: simulation/aws-robomaker-sample-application-deepracer/simulation_ws/src/deepracer_simulation/urdf/mit/racecar.xacro (robot description, xacro)
@@ -1,5 +1,7 @@
 <?xml version="1.0"?>
 <robot name="racecar" xmlns:xacro="http://www.ros.org/wiki/xacro">
-  <xacro:include filename="$(find deepracer_simulation)/urdf/macros.xacro" />
+  <xacro:include filename="$(find deepracer_simulation)/urdf/mit/macros.xacro" />
+  <xacro:arg name="include_second_camera" default="false" />
+  <xacro:arg name="include_lidar_sensor" default="false" />
   <!-- Add chassis and it's inertia link -->
   <link name="base_link" />
@@ -202,5 +204,5 @@
   </joint>
   <!-- Add the remaining xacros -->
-  <xacro:include filename="$(find deepracer_simulation)/urdf/racecar.gazebo" />
-  <xacro:include filename="$(find deepracer_simulation)/urdf/materials.xacro" />
+  <xacro:include filename="$(find deepracer_simulation)/urdf/mit/racecar.gazebo" />
+  <xacro:include filename="$(find deepracer_simulation)/urdf/mit/materials.xacro" />
 </robot>
